File: HardwareSystem/Probe/PCB_Probe/PCB_Probe/_autosave-PCB_Probe.kicad_sch (KiCad schematic)
At the start: 7 parts, among them U1 TLC555xP

Commit message: PCB probe WIP
Parts:
- added A2: Arduino_Nano_v3.x, Module:Arduino_Nano, symbol MCU_Module:Arduino_Nano_v3.x
- added BT1: Battery, symbol Device:Battery
- added C4: 10u, Capacitor_THT:C_Disc_D3.0mm_W1.6mm_P2.50mm, symbol Device:C
- added C5, C7: 4.7u, Capacitor_THT:C_Disc_D3.0mm_W1.6mm_P2.50mm, symbol Device:C
- added C6, C8: 100n, Capacitor_THT:C_Disc_D3.0mm_W1.6mm_P2.50mm, symbol Device:C
- added D1: 1N4148WS, Diode_SMD:D_SOD-323, symbol Diode:1N4148WS
- added R4: 1M, Resistor_THT:R_Axial_DIN0204_L3.6mm_D1.6mm_P5.08mm_Horizontal, symbol Device:R
- added U2: XC6206PxxxMR, Package_TO_SOT_SMD:SOT-23-3, symbol Regulator_Linear:XC6206PxxxMR
- C1, C2: footprint (none) -> Capacitor_THT:C_Disc_D3.0mm_W1.6mm_P2.50mm
- C3: value 460pF -> 470pF; footprint (none) -> Capacitor_THT:C_Disc_D3.0mm_W1.6mm_P2.50mm
- R1, R2, R3: footprint (none) -> Resistor_THT:R_Axial_DIN0204_L3.6mm_D1.6mm_P5.08mm_Horizontal
Connections:
- net +3.3V: now also C5.1, C6.1, U2.3 (VI); no longer C1.1, R1.1, U1.4 (R), U1.8 (VCC)
- net GND: now also C1.1, C3.1, R3.2, C4.2, C5.2, C6.2, C7.2, C8.2, D1.2 (A), R4.1, U2.1 (GND); no longer C1.2, C3.2
- net at U1.2 (TR), U1.6 (THR): now also C3.2, R2.1; no longer C3.1, R2.2
- net at R1.2, U1.7 (DIS): now also R2.2; no longer R2.1
- new net +3V0: C1.2, C7.1, C8.1, R1.1, U1.4 (R), U1.8 (VCC), U2.2 (VO)
- new net MOut: C4.1, D1.1 (K), R4.2
Other:
- note added: "3.3V to 3V LDO"
- note added: "Arduino Nano ESP32"
- note added: "Capactive Moisture Sensor"
- title: (none) -> APWS-SP10-HW-Probe
- moved on the sheet: U1
