File: HardwareSystem/Probe/PCB_Probe/PCB_Probe/PCB_Probe.kicad_sch (KiCad schematic)
At the start: 15 parts, among them U1 TLC555xP, U2 XC6206PxxxMR

Commit message: Added more circuits to PCB probe
Added more circuits to PCB probe
Parts:
- removed C5: 4.7u, symbol Device:C
- removed C8: 100n, symbol Device:C
- removed U2: XC6206PxxxMR, Package_TO_SOT_SMD:SOT-23-3, symbol Regulator_Linear:XC6206PxxxMR
- added A2: Arduino_Nano_v3.x, Module:Arduino_Nano, symbol MCU_Module:Arduino_Nano_v3.x
- added BT1: BH9VPC, BH9VPC:BAT_BH9VPC, symbol BH9VPC:BH9VPC
- added C10, C9: 100nF, Capacitor_THT:C_Disc_D3.0mm_W1.6mm_P2.50mm, symbol Device:C
- added J1, J2: Conn_01x15, Connector_PinSocket_1.00mm:PinSocket_1x15_P1.00mm_Vertical, symbol Connector_Generic:Conn_01x15
- added R6: 10kR, Resistor_THT:R_Axial_DIN0204_L3.6mm_D1.6mm_P5.08mm_Horizontal, symbol Device:R
- added R7: Photoresistor, KiCADv6:XDCR_161, symbol 161:Photoresistor
- added TP1: 5V Testpoint, TestPoint:TestPoint_Pad_D1.0mm, symbol Connector:TestPoint
- added TP2: 3.3V Testpoint, TestPoint:TestPoint_Pad_D1.0mm, symbol Connector:TestPoint
- added TP3: 3V Testpoint, TestPoint:TestPoint_Pad_D1.0mm, symbol Connector:TestPoint
- added U2: LP2950CZ-3.0/NOPB, Z03A_TEX, symbol 2024-02-28_23-11-38:LP2950CZ-3.0_NOPB
- C1: value 100n -> 100nF; footprint (none) -> Capacitor_THT:C_Disc_D3.0mm_W1.6mm_P2.50mm
- C2: value 10n -> 10nF; footprint (none) -> Capacitor_THT:C_Disc_D3.0mm_W1.6mm_P2.50mm
- C3: footprint (none) -> Capacitor_THT:C_Disc_D3.0mm_W1.6mm_P2.50mm
- C4: value 10u -> 10uF; footprint (none) -> Capacitor_THT:C_Disc_D3.0mm_W1.6mm_P2.50mm
- C5: renamed from C6; value 100n -> 4.7uF; footprint (none) -> Capacitor_THT:C_Disc_D3.0mm_W1.6mm_P2.50mm
- C6: renamed from C7; value 4.7u -> 1uF; footprint (none) -> Capacitor_THT:C_Disc_D3.0mm_W1.6mm_P2.50mm
- R1: value 330 -> 330R; footprint (none) -> Resistor_THT:R_Axial_DIN0204_L3.6mm_D1.6mm_P5.08mm_Horizontal
- R2: value 1.6k -> 1.6kR; footprint (none) -> Resistor_THT:R_Axial_DIN0204_L3.6mm_D1.6mm_P5.08mm_Horizontal
- R3: value 10k -> 10kR; footprint (none) -> Resistor_THT:R_Axial_DIN0204_L3.6mm_D1.6mm_P5.08mm_Horizontal
- R4: value 1M -> 1MF; footprint (none) -> Resistor_THT:R_Axial_DIN0204_L3.6mm_D1.6mm_P5.08mm_Horizontal
Connections:
- net +3.3V: now also A2.17 (3V3), J1.2 (Pin_2), J1.5 (Pin_5), R7.1, TP2.1, U2.1 (OUT)
- net +3V0: now also TP3.1, U2.3 (IN)
- net GND: now also A2.29 (GND), A2.4 (GND), BT1.-, C10.2, C9.2, J2.12 (Pin_12), R6.1, U2.2 (GND)
- net MOut renamed A_Moisture
- net A_Moisture: now also J1.4 (Pin_4)
- new net: R6.2, R7.2
- new net +9V: A2.30 (VIN), BT1.+, C10.1, C9.1, J1.15 (Pin_15), TP1.1
- new net SCL: J1.9 (Pin_9)
- new net SDA: J1.8 (Pin_8)
Other:
- note added: "9V Battery"
- note added: "Arduino Nano ESP32"
- note added: "Arduino headers"
- note added: "Capactive Moisture Sensor"
- note added: "D12 D11 D10 D9 D8 D7 D6 D5 D4 D2 D1 GND RST RX0 TX1"
- note added: "D13 3.3V B0 A0 A1 A2 A3 A4 A5 A6 A7 VBUS B1 GND VIN"
- note added: "DNP"
- note added: "Decoupling Caps"
- note added: "Photoresistor"
- title: (none) -> APWS-SP10-HW-Probe
- moved on the sheet: C1, C2, C3, C4, C5, C6, D1, R1, R2, R3, R4, U1
