File: HardwareSystem/Probe/PCB_Pump/PCB_Pump/PCB_Pump.kicad_pcb (KiCad board)
At the start: 2 copper layers, 20.8 x 66.8 mm, 4 parts, among them Q1 IRF510

Commit message: pump pcb work
Parts:
- removed A1: Arduino_Nano_Every, Module:Arduino_Nano
- added +: PinHeader_1x02_P2.54mm_Vertical, Connector_PinHeader_2.54mm:PinHeader_1x02_P2.54mm_Vertical, F.Cu at (169.2, 42.9)
- added A2: Arduino_Nano_ESP32_Socket, footprints:Arduino_Nano_ESP32_Socket, F.Cu at (155.7, 84.1)
- added C1: 0.1 uF, Capacitor_THT:C_Axial_L3.8mm_D2.6mm_P7.50mm_Horizontal, F.Cu at (167.6, 51.1)
- added C2: 10 uF, Capacitor_THT:C_Axial_L5.1mm_D3.1mm_P7.50mm_Horizontal, F.Cu at (173.7, 51.1)
- added REF**: MountingHole_2.1mm, MountingHole:MountingHole_2.1mm, F.Cu at (179.8, 43.4)
- added REF**: MountingHole_2.1mm, MountingHole:MountingHole_2.1mm, F.Cu at (144.0, 43.4)
- added REF**: MountingHole_2.1mm, MountingHole:MountingHole_2.1mm, F.Cu at (179.8, 81.5)
- added REF**: MountingHole_2.1mm, MountingHole:MountingHole_2.1mm, F.Cu at (144.0, 81.5)
- added TP5V: TestPoint_Keystone_5000-5004_Miniature, TestPoint:TestPoint_Keystone_5000-5004_Miniature, F.Cu at (168.7, 63.2)
- added U1: LM2937xT, Package_TO_SOT_THT:TO-220-3_Vertical, F.Cu at (167.9, 48.1)
- added p+: PinHeader_1x02_P2.54mm_Vertical, Connector_PinHeader_2.54mm:PinHeader_1x02_P2.54mm_Vertical, F.Cu at (175.5, 70.1)
- moved D1 32.4 mm to (171.7, 67.6), turned to -90 degrees
- moved R1 28.1 mm to (168.7, 67.6), turned to -90 degrees
- moved Q1 14.3 mm to (168.7, 79.0), turned to 0 degrees
Routing:
- net GND: track 18.0 -> 51.4 mm, vias 0 -> 1
- net Net-(A2-PadD8): track 53.3 -> 21.6 mm
- net pump+: track 0.00 -> 29.7 mm, vias 0 -> 2
- net 9V: track 0.00 -> 16.7 mm
- net Net-(Q1-G): track 6.79 -> 3.83 mm
- net pump-: track 5.91 -> 8.82 mm
Other:
- board size 20.8 x 66.8 mm -> 40.9 x 43.2 mm
- board text added: "-"
- board text added: "p-"

Commit message: finished PCB pump
Parts:
- moved D1 39.4 mm to (145.3, 96.7)
- moved Q1 39.4 mm to (142.3, 108.2)
- moved R1 39.4 mm to (142.2, 96.7)
- moved p+ 39.4 mm to (149.1, 99.3)
- moved TP5V 39.4 mm to (142.2, 92.4)
- moved REF** 39.4 mm to (117.6, 72.6)
- moved REF** 39.4 mm to (117.6, 110.7)
- moved + 39.4 mm to (142.7, 72.1)
- moved A2 39.4 mm to (129.3, 113.3)
- moved C1 39.4 mm to (141.2, 80.2)
- moved C2 39.4 mm to (147.3, 80.2)
- moved REF** 39.4 mm to (153.4, 72.6)
- moved REF** 39.4 mm to (153.4, 110.7)
- moved U1 39.4 mm to (141.5, 77.3)
Other:
- board text added: "APWS-SP10 Alexis Torres, Evan LeBel, Ian Skillman, Jaime Sanchez, Javier Padilla, Jesus Hernandez, Kiet Le, Rodrigo Romero"
- board text removed: "notes: center it put mounting holes don't put wires under the arduino - wifi/ble here"

Commit message: pcb pump revision
Parts:
- added GND: Conn_01x04_Pin, Connector_PinHeader_2.54mm:PinHeader_1x04_P2.54mm_Vertical, F.Cu at (118.1, 89.1)
- moved p+ 4.34 mm to (153.4, 99.3)
Connections:
- A2 pad D2: unconnected-(A2-PadD2) -> Trig
- A2 pad D3: unconnected-(A2-PadD3) -> Echo
- A2 pad GND2: GND -> Net-(A2-GND-PadGND1)
Routing:
- net pump+: track 29.7 -> 70.4 mm, vias 2 -> 3
- net GND: track 51.4 -> 68.7 mm, vias 1 -> 2
- net pump-: track 8.82 -> 13.1 mm
- net Trig: track 0.00 -> 3.56 mm
- net Echo: track 0.00 -> 3.56 mm
Other:
- outline, holes or cut-outs redrawn
- board text added: "VCC"

Commit message: pumpv2-v3
Connections:
- A2 pad GND2: Net-(A2-GND-PadGND1) -> GND
Other:
- board size 40.9 x 43.2 mm -> 40.9 x 44.7 mm
Changed lines of the file:
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@@
   (net 31 "unconnected-(A2-Pad5V)")
   (net 32 "9V")
-  (net 33 "Net-(A2-GND-PadGND1)")
   (footprint "Connector_PinHeader_2.54mm:PinHeader_1x02_P2.54mm_Vertical" (layer "F.Cu")
     (at 153.416 99.309)
@@
     (tags "mounting hole 2.1mm no annular")
     (attr exclude_from_pos_files exclude_from_bom)
-    (fp_text reference "REF**" (at 0 -3.2) (layer "F.SilkS")
+    (fp_text reference "REF**" (at 0 -3.2) (layer "F.SilkS") hide
         (effects (font (size 1 1) (thickness 0.15)))
     )
@@
     (tags "mounting hole 2.1mm no annular")
     (attr exclude_from_pos_files exclude_from_bom)
-    (fp_text reference "REF**" (at 0 -3.2) (layer "F.SilkS")
+    (fp_text reference "REF**" (at 0 -3.2) (layer "F.SilkS") hide
         (effects (font (size 1 1) (thickness 0.15)))
     )
@@
     (property "ki_description" "MOSFET RECOMMENDED ALT 844-IRF510PBF")
     (attr through_hole)
-    (fp_text reference "Q1" (at -0.35 0 unlocked) (layer "B.SilkS")
+    (fp_text reference "Q1" (at -0.031 1.8107 unlocked) (layer "B.SilkS")
         (effects (font (size 1 1) (thickness 0.15)) (justify mirror))
     )
@@
     (property "ki_keywords" "Arduino MPU Shield")
     (attr through_hole)
-    (fp_text reference "A2" (at 0 -44.45) (layer "F.SilkS")
+    (fp_text reference "A2" (at 0 -42.164) (layer "F.SilkS")
         (effects (font (size 1 1) (thickness 0.15)))
     )
@@
       (net 3 "GND") (pinfunction "GND") (pintype "power_in"))
     (pad "GND2" thru_hole rect (at 7.62 -36.83) (size 1.7272 1.7272) (drill 1.016) (layers "*.Cu" "*.Mask")
-      (net 33 "Net-(A2-GND-PadGND1)") (pinfunction "GND") (pintype "power_in"))
+      (net 3 "GND") (pinfunction "GND") (pintype "power_in"))
     (pad "RST" thru_hole circle (at -7.62 -34.29) (size 1.7272 1.7272) (drill 1.016) (layers "*.Cu" "*.Mask")
       (net 30 "unconnected-(A2-~{RESET}-PadRST)") (pinfunction "~{RESET}") (pintype "open_collector"))
@@
     (pad "" np_thru_hole circle (at 0 0) (size 2.1 2.1) (drill 2.1) (layers "F&B.Cu" "*.Mask"))
   )
-  (gr_arc (start 115.038999 70.866) (mid 115.255166 70.320167) (end 115.800999 70.104)
-    (stroke (width 0.15) (type default)) (layer "Edge.Cuts"))
-  (gr_line (start 155.932999 108.1713) (end 155.932999 75.1513)
-    (stroke (width 0.15) (type default)) (layer "Edge.Cuts"))
-  (gr_line (start 115.800999 70.104) (end 155.170999 70.104)
-    (stroke (width 0.15) (type default)) (layer "Edge.Cuts"))
-  (gr_line (start 115.038999 70.866) (end 115.038999 75.1513)
-    (stroke (width 0.15) (type default)) (layer "Edge.Cuts"))
-  (gr_line (start 115.038999 108.1713) (end 115.038999 112.522)
-    (stroke (width 0.15) (type default)) (layer "Edge.Cuts"))
-  (gr_line (start 155.932999 108.1713) (end 155.918167 112.484167)
+  (gr_arc (start 115.038999 70.104) (mid 115.267481 69.570482) (end 115.800999 69.342)
+    (stroke (width 0.15) (type default)) (layer "Edge.Cuts"))
+  (gr_line (start 155.956 113.265083) (end 155.956 70.104)
+    (stroke (width 0.15) (type default)) (layer "Edge.Cuts"))
+  (gr_line (start 115.800999 69.342) (end 155.194 69.342)
+    (stroke (width 0.15) (type default)) (layer "Edge.Cuts"))
+  (gr_line (start 115.038999 70.104) (end 115.038999 75.1513)
+    (stroke (width 0.15) (type default)) (layer "Edge.Cuts"))
+  (gr_arc (start 155.956 113.265083) (mid 155.727518 113.798601) (end 155.194 114.027083)
+    (stroke (width 0.15) (type default)) (layer "Edge.Cuts"))
+  (gr_arc (start 155.194 69.342) (mid 155.727518 69.570482) (end 155.956 70.104)
+    (stroke (width 0.15) (type default)) (layer "Edge.Cuts"))
+  (gr_line (start 115.038999 108.1713) (end 115.038999 113.302916)
     (stroke (width 0.15) (type default)) (layer "Edge.Cuts"))
   (gr_line (start 115.038999 75.1513) (end 115.038999 108.1713)
     (stroke (width 0.15) (type default)) (layer "Edge.Cuts"))
-  (gr_arc (start 115.800999 113.284) (mid 115.255166 113.067833) (end 115.038999 112.522)
-    (stroke (width 0.15) (type default)) (layer "Edge.Cuts"))
-  (gr_line (start 115.800999 113.284) (end 155.156167 113.246167)
-    (stroke (width 0.15) (type default)) (layer "Edge.Cuts"))
-  (gr_arc (start 155.170999 70.104) (mid 155.716832 70.320167) (end 155.932999 70.866)
-    (stroke (width 0.15) (type default)) (layer "Edge.Cuts"))
-  (gr_line (start 155.932999 70.866) (end 155.932999 75.1513)
-    (stroke (width 0.15) (type default)) (layer "Edge.Cuts"))
-  (gr_arc (start 155.918167 112.484167) (mid 155.702 113.03) (end 155.156167 113.246167)
+  (gr_line (start 115.800999 114.064916) (end 155.194 114.027083)
+    (stroke (width 0.15) (type default)) (layer "Edge.Cuts"))
+  (gr_arc (start 115.800999 114.064916) (mid 115.267481 113.836434) (end 115.038999 113.302916)
     (stroke (width 0.15) (type default)) (layer "Edge.Cuts"))
   (gr_text "VCC" (at 118.11 79.248) (layer "F.SilkS")
